File: kicad/projeto/projeto.kicad_sch (KiCad schematic)
At the start: 40 parts, among them Q1 BTA16-600B, Q2 BTA16-600B, U1 ESP-12E, U3v3 LM1117-3.3

Commit message: Att componentes
Parts:
- removed Uload1, Uload2: MOC3023M, Package_DIP:DIP-6_W7.62mm_Socket, symbol Relay_SolidState:MOC3021M
- added Uload1, Uload2: MOC3023M, Package_DIP:DIP-6_W7.62mm_LongPads, symbol Relay_SolidState:MOC3023M
- D5: value 5V -> 7.5V; footprint (none) -> Diode_THT:D_T-1_P5.08mm_Horizontal
- Ren1: value 33K -> 10K
- Rz1: footprint Resistor_THT:R_Axial_DIN0207_L6.3mm_D2.5mm_P10.16mm_Horizontal -> Resistor_THT:R_Axial_DIN0309_L9.0mm_D3.2mm_P12.70mm_Horizontal
Connections:
- net GND: now also Uload1.4, Uload2.4
- net at Rtriac1.1: now also Uload1.1
- net at Rmoc1.1: now also Uload1.6
- net at Q1.3 (G): now also Uload1.2
- net at Rtriac2.1: now also Uload2.1
- net at Rmoc2.1: now also Uload2.6
- net at Q2.3 (G): now also Uload2.2
Changed lines of the file:
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@@
     (effects (font (size 1.27 1.27)) (justify left bottom))
   )
-  (text "Power" (at 176.53 118.11 0)
+  (text "Power" (at 231.14 118.11 0)
     (effects (font (size 1.27 1.27)) (justify left bottom))
   )
@@
     (pin "2")
   )
-  (symbol (lib_id "Relay_SolidState:MOC3021M") (at 85.09 140.97 0) (mirror y) (unit 1)
-    (in_bom yes) (on_board yes)
-    (property "Reference" "Uload1" (id 0) (at 85.09 132.08 0))
-    (property "Value" "MOC3023M" (id 1) (at 85.09 134.62 0))
-    (property "Footprint" "Package_DIP:DIP-6_W7.62mm_Socket" (id 2) (at 90.17 146.05 0)
-      (effects (font (size 1.27 1.27) italic) (justify left) hide)
-    )
-    (property "Datasheet" "https://www.onsemi.com/pub/Collateral/MOC3023M-D.PDF" (id 3) (at 85.09 140.97 0)
-      (effects (font (size 1.27 1.27)) (justify left) hide)
-    )
-    (pin "1")
-    (pin "2")
-    (pin "3")
-    (pin "4")
-    (pin "5")
-    (pin "6")
-  )
   (symbol (lib_id "Diode:UF5408") (at 101.6 91.44 270) (unit 1)
     (in_bom yes) (on_board yes) (fields_autoplaced)
@@
     (pin "1")
   )
+  (symbol (lib_id "Relay_SolidState:MOC3023M") (at 85.09 171.45 0) (unit 1)
+    (in_bom yes) (on_board yes) (fields_autoplaced)
+    (property "Reference" "Uload2" (id 0) (at 85.09 162.56 0))
+    (property "Value" "MOC3023M" (id 1) (at 85.09 165.1 0))
+    (property "Footprint" "Package_DIP:DIP-6_W7.62mm_LongPads" (id 2) (at 80.01 176.53 0)
+      (effects (font (size 1.27 1.27) italic) (justify left) hide)
+    )
+    (property "Datasheet" "https://www.onsemi.com/pub/Collateral/MOC3023M-D.PDF" (id 3) (at 85.09 171.45 0)
+      (effects (font (size 1.27 1.27)) (justify left) hide)
+    )
+    (pin "1")
+    (pin "2")
+    (pin "3")
+    (pin "4")
+    (pin "5")
+    (pin "6")
+  )
   (symbol (lib_id "power:+3V3") (at 46.99 90.17 0) (unit 1)
     (in_bom yes) (on_board yes) (fields_autoplaced)
@@
       (effects (font (size 1.27 1.27)) (justify right))
     )
-    (property "Value" "33K" (id 1) (at 189.23 54.6099 0)
+    (property "Value" "10K" (id 1) (at 189.23 54.6099 0)
       (effects (font (size 1.27 1.27)) (justify right))
     )
@@
     (property "Reference" "Rz1" (id 0) (at 127 91.44 90))
     (property "Value" "33k" (id 1) (at 127 93.98 90))
-    (property "Footprint" "Resistor_THT:R_Axial_DIN0207_L6.3mm_D2.5mm_P10.16mm_Horizontal" (id 2) (at 124.46 98.298 90)
+    (property "Footprint" "Resistor_THT:R_Axial_DIN0309_L9.0mm_D3.2mm_P12.70mm_Horizontal" (id 2) (at 124.46 98.298 90)
       (effects (font (size 1.27 1.27)) hide)
     )
@@
     )
     (pin "1")
+  )
+  (symbol (lib_id "Relay_SolidState:MOC3023M") (at 85.09 140.97 0) (unit 1)
+    (in_bom yes) (on_board yes) (fields_autoplaced)
+    (property "Reference" "Uload1" (id 0) (at 85.09 132.08 0))
+    (property "Value" "MOC3023M" (id 1) (at 85.09 134.62 0))
+    (property "Footprint" "Package_DIP:DIP-6_W7.62mm_LongPads" (id 2) (at 80.01 146.05 0)
+      (effects (font (size 1.27 1.27) italic) (justify left) hide)
+    )
+    (property "Datasheet" "https://www.onsemi.com/pub/Collateral/MOC3023M-D.PDF" (id 3) (at 85.09 140.97 0)
+      (effects (font (size 1.27 1.27)) (justify left) hide)
+    )
+    (pin "1")
+    (pin "2")
+    (pin "3")
+    (pin "4")
+    (pin "5")
+    (pin "6")
   )
   (symbol (lib_id "power:GND") (at 123.19 64.77 0) (unit 1)
@@
     )
     (pin "1")
-  )
-  (symbol (lib_id "Relay_SolidState:MOC3021M") (at 85.09 171.45 0) (mirror y) (unit 1)
-    (in_bom yes) (on_board yes)
-    (property "Reference" "Uload2" (id 0) (at 85.09 162.56 0))
-    (property "Value" "MOC3023M" (id 1) (at 85.09 165.1 0))
-    (property "Footprint" "Package_DIP:DIP-6_W7.62mm_Socket" (id 2) (at 90.17 176.53 0)
-      (effects (font (size 1.27 1.27) italic) (justify left) hide)
-    )
-    (property "Datasheet" "https://www.onsemi.com/pub/Collateral/MOC3023M-D.PDF" (id 3) (at 85.09 171.45 0)
-      (effects (font (size 1.27 1.27)) (justify left) hide)
-    )
-    (pin "1")
-    (pin "2")
-    (pin "3")
-    (pin "4")
-    (pin "5")
-    (pin "6")
   )
   (symbol (lib_id "power:+3V3") (at 73.66 34.29 0) (unit 1)
@@
     (in_bom yes) (on_board yes) (fields_autoplaced)
     (property "Reference" "D5" (id 0) (at 116.84 90.17 0))
-    (property "Value" "5V" (id 1) (at 116.84 92.71 0))
-    (property "Footprint" "" (id 2) (at 116.84 96.52 0)
+    (property "Value" "7.5V" (id 1) (at 116.84 92.71 0))
+    (property "Footprint" "Diode_THT:D_T-1_P5.08mm_Horizontal" (id 2) (at 116.84 96.52 0)
       (effects (font (size 1.27 1.27)) hide)
     )
@@
     )
     (path "/e483a1a3-bb43-4adf-8c54-28292661b80b"
-      (reference "D5") (unit 1) (value "5V") (footprint "")
+      (reference "D5") (unit 1) (value "7.5V") (footprint "Diode_THT:D_T-1_P5.08mm_Horizontal")
     )
     (path "/3abfc083-ebde-48d2-8837-cffffdca55ee"
@@
     )
     (path "/5620de57-8f1e-490c-b1e4-fcb9f7a57928"
-      (reference "Ren1") (unit 1) (value "33K") (footprint "Resistor_THT:R_Axial_DIN0207_L6.3mm_D2.5mm_P7.62mm_Horizontal")
+      (reference "Ren1") (unit 1) (value "10K") (footprint "Resistor_THT:R_Axial_DIN0207_L6.3mm_D2.5mm_P7.62mm_Horizontal")
     )
     (path "/55eb4026-97a3-4a48-9280-a37bc89991bd"
@@
     )
     (path "/71c6153a-0b50-4d67-b5e3-af65b0c1027f"
-      (reference "Rz1") (unit 1) (value "33k") (footprint "Resistor_THT:R_Axial_DIN0207_L6.3mm_D2.5mm_P10.16mm_Horizontal")
+      (reference "Rz1") (unit 1) (value "33k") (footprint "Resistor_THT:R_Axial_DIN0309_L9.0mm_D3.2mm_P12.70mm_Horizontal")
     )
     (path "/a43a8617-6998-45ef-aaca-a374304030fe"
@@
       (reference "Udet_0") (unit 1) (value "4N25") (footprint "Package_DIP:DIP-6_W7.62mm")
     )
-    (path "/0b7062df-746f-4e3d-8ab7-859629a51a0d"
-      (reference "Uload1") (unit 1) (value "MOC3023M") (footprint "Package_DIP:DIP-6_W7.62mm_Socket")
-    )
-    (path "/a92d2b21-44f0-4225-aa43-a193282d0dbd"
-      (reference "Uload2") (unit 1) (value "MOC3023M") (footprint "Package_DIP:DIP-6_W7.62mm_Socket")
+    (path "/8cfda358-272c-4e6e-87ec-7984a71789c0"
+      (reference "Uload1") (unit 1) (value "MOC3023M") (footprint "Package_DIP:DIP-6_W7.62mm_LongPads")
+    )
+    (path "/20b388b4-d21d-4e6e-aa24-541e239049a3"
+      (reference "Uload2") (unit 1) (value "MOC3023M") (footprint "Package_DIP:DIP-6_W7.62mm_LongPads")
     )
     (path "/9e0b94a4-21da-4ce8-89a2-32c3571760d1"

Commit message: Fazendo a PCB (1)
Parts:
- removed Jdc1: Barrel_Jack_MountingPin, Connector_BarrelJack:BarrelJack_Horizontal, symbol Connector:Barrel_Jack_MountingPin
- added Jdc1: Barrel_Jack_Switch, Connector_BarrelJack:BarrelJack_CUI_PJ-102AH_Horizontal, symbol Connector:Barrel_Jack_Switch
- D1, D2, D3, D4: footprint Diode_THT:D_DO-201AD_P15.24mm_Horizontal -> Diode_THT:D_T-1_P5.08mm_Horizontal
Connections:
- net +5V: now also Jdc1.1
- net GND: now also Jdc1.2
- net at D2.2 (A), D4.2 (A): now also Rz1.2; no longer Udet_0.2
- net at Udet_0.1: now also D5.2 (A); no longer Rz1.2
- net at Rz1.1: now also Udet_0.2; no longer D5.2 (A)
Other:
- moved on the sheet: Rz1
Changed lines of the file:
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@@
+    (stroke (width 0) (type default) (color 0 0 0 0))
+  )
+  (wire (pts (xy 133.35 142.24) (xy 132.08 142.24))
     (stroke (width 0) (type default) (color 0 0 0 0))
   )
@@
     (stroke (width 0) (type default) (color 0 0 0 0))
   )
+  (wire (pts (xy 133.35 147.32) (xy 124.46 147.32))
+    (stroke (width 0) (type default) (color 0 0 0 0))
+  )
   (polyline (pts (xy 110.49 115.57) (xy 237.49 115.57))
     (stroke (width 0) (type default) (color 0 0 0 0))
@@
     (stroke (width 0) (type default) (color 0 0 0 0))
   )
+  (wire (pts (xy 125.73 101.6) (xy 128.27 101.6))
+    (stroke (width 0) (type default) (color 0 0 0 0))
+  )
   (wire (pts (xy 143.51 99.06) (xy 151.13 99.06))
     (stroke (width 0) (type default) (color 0 0 0 0))
@@
     (stroke (width 0) (type default) (color 0 0 0 0))
   )
+  (wire (pts (xy 133.35 142.24) (xy 133.35 147.32))
+    (stroke (width 0) (type default) (color 0 0 0 0))
+  )
   (wire (pts (xy 92.71 168.91) (xy 95.25 168.91))
     (stroke (width 0) (type default) (color 0 0 0 0))
@@
     (stroke (width 0) (type default) (color 0 0 0 0))
   )
-  (wire (pts (xy 124.46 152.4) (xy 124.46 149.86))
+  (wire (pts (xy 124.46 147.32) (xy 124.46 152.4))
     (stroke (width 0) (type default) (color 0 0 0 0))
   )
@@
     (stroke (width 0) (type default) (color 0 0 0 0))
   )
-  (wire (pts (xy 101.6 101.6) (xy 128.27 101.6))
+  (wire (pts (xy 101.6 101.6) (xy 118.11 101.6))
     (stroke (width 0) (type default) (color 0 0 0 0))
   )
@@
   )
   (wire (pts (xy 213.36 133.35) (xy 210.82 133.35))
+    (stroke (width 0) (type default) (color 0 0 0 0))
+  )
+  (wire (pts (xy 120.65 96.52) (xy 128.27 96.52))
     (stroke (width 0) (type default) (color 0 0 0 0))
   )
@@
       (effects (font (size 1.27 1.27)) (justify left))
     )
-    (property "Footprint" "Diode_THT:D_DO-201AD_P15.24mm_Horizontal" (id 2) (at 84.455 106.68 0)
+    (property "Footprint" "Diode_THT:D_T-1_P5.08mm_Horizontal" (id 2) (at 84.455 106.68 0)
       (effects (font (size 1.27 1.27)) hide)
     )
@@
       (effects (font (size 1.27 1.27)) (justify left))
     )
-    (property "Footprint" "Diode_THT:D_DO-201AD_P15.24mm_Horizontal" (id 2) (at 97.155 91.44 0)
+    (property "Footprint" "Diode_THT:D_T-1_P5.08mm_Horizontal" (id 2) (at 97.155 91.44 0)
       (effects (font (size 1.27 1.27)) hide)
     )
@@
       (effects (font (size 1.27 1.27)) (justify right))
     )
-    (property "Footprint" "Diode_THT:D_DO-201AD_P15.24mm_Horizontal" (id 2) (at 93.345 91.44 0)
+    (property "Footprint" "Diode_THT:D_T-1_P5.08mm_Horizontal" (id 2) (at 93.345 91.44 0)
       (effects (font (size 1.27 1.27)) hide)
     )
@@
     (pin "1")
   )
-  (symbol (lib_id "Device:R") (at 124.46 96.52 90) (unit 1)
+  (symbol (lib_id "Device:R") (at 121.92 101.6 270) (unit 1)
     (in_bom yes) (on_board yes)
-    (property "Reference" "Rz1" (id 0) (at 127 91.44 90))
-    (property "Value" "33k" (id 1) (at 127 93.98 90))
-    (property "Footprint" "Resistor_THT:R_Axial_DIN0309_L9.0mm_D3.2mm_P12.70mm_Horizontal" (id 2) (at 124.46 98.298 90)
-      (effects (font (size 1.27 1.27)) hide)
-    )
-    (property "Datasheet" "~" (id 3) (at 124.46 96.52 0)
+    (property "Reference" "Rz1" (id 0) (at 119.38 106.68 90))
+    (property "Value" "33k" (id 1) (at 119.38 104.14 90))
+    (property "Footprint" "Resistor_THT:R_Axial_DIN0309_L9.0mm_D3.2mm_P12.70mm_Horizontal" (id 2) (at 121.92 99.822 90)
+      (effects (font (size 1.27 1.27)) hide)
+    )
+    (property "Datasheet" "~" (id 3) (at 121.92 101.6 0)
       (effects (font (size 1.27 1.27)) hide)
     )
@@
       (effects (font (size 1.27 1.27)) (justify right))
     )
-    (property "Footprint" "Diode_THT:D_DO-201AD_P15.24mm_Horizontal" (id 2) (at 106.045 106.68 0)
+    (property "Footprint" "Diode_THT:D_T-1_P5.08mm_Horizontal" (id 2) (at 106.045 106.68 0)
       (effects (font (size 1.27 1.27)) hide)
     )
@@
     )
     (pin "1")
-  )
-  (symbol (lib_id "Connector:Barrel_Jack_MountingPin") (at 124.46 142.24 0) (unit 1)
-    (in_bom yes) (on_board yes) (fields_autoplaced)
-    (property "Reference" "Jdc1" (id 0) (at 124.46 133.35 0))
-    (property "Value" "Barrel_Jack_MountingPin" (id 1) (at 124.46 135.89 0))
-    (property "Footprint" "Connector_BarrelJack:BarrelJack_Horizontal" (id 2) (at 125.73 143.256 0)
-      (effects (font (size 1.27 1.27)) hide)
-    )
-    (property "Datasheet" "~" (id 3) (at 125.73 143.256 0)
-      (effects (font (size 1.27 1.27)) hide)
-    )
-    (pin "1")
-    (pin "2")
-    (pin "MP")
   )
   (symbol (lib_id "Device:R") (at 151.13 93.98 0) (unit 1)
@@
     (pin "9")
   )
+  (symbol (lib_id "Connector:Barrel_Jack_Switch") (at 124.46 142.24 0) (unit 1)
+    (in_bom yes) (on_board yes) (fields_autoplaced)
+    (property "Reference" "Jdc1" (id 0) (at 124.46 133.35 0))
+    (property "Value" "Barrel_Jack_Switch" (id 1) (at 124.46 135.89 0))
+    (property "Footprint" "Connector_BarrelJack:BarrelJack_CUI_PJ-102AH_Horizontal" (id 2) (at 125.73 143.256 0)
+      (effects (font (size 1.27 1.27)) hide)
+    )
+    (property "Datasheet" "~" (id 3) (at 125.73 143.256 0)
+      (effects (font (size 1.27 1.27)) hide)
+    )
+    (pin "1")
+    (pin "2")
+    (pin "3")
+  )
   (symbol (lib_id "Triac_Thyristor:BTA16-600B") (at 64.77 171.45 0) (mirror y) (unit 1)
     (in_bom yes) (on_board yes)
@@
     )
     (path "/6c7ba7e5-1a29-4616-9eaf-31ecc6a51cb4"
-      (reference "D1") (unit 1) (value "UF5408") (footprint "Diode_THT:D_DO-201AD_P15.24mm_Horizontal")
+      (reference "D1") (unit 1) (value "UF5408") (footprint "Diode_THT:D_T-1_P5.08mm_Horizontal")
     )
     (path "/0d328538-f690-4df1-aec5-07d7902549d3"
-      (reference "D2") (unit 1) (value "UF5408") (footprint "Diode_THT:D_DO-201AD_P15.24mm_Horizontal")
+      (reference "D2") (unit 1) (value "UF5408") (footprint "Diode_THT:D_T-1_P5.08mm_Horizontal")
     )
     (path "/04bfdb7a-c251-4427-8798-e9028c17447a"
-      (reference "D3") (unit 1) (value "UF5408") (footprint "Diode_THT:D_DO-201AD_P15.24mm_Horizontal")
+      (reference "D3") (unit 1) (value "UF5408") (footprint "Diode_THT:D_T-1_P5.08mm_Horizontal")
     )
     (path "/7a4d805a-3f12-425f-be61-714f86901361"
-      (reference "D4") (unit 1) (value "UF5408") (footprint "Diode_THT:D_DO-201AD_P15.24mm_Horizontal")
+      (reference "D4") (unit 1) (value "UF5408") (footprint "Diode_THT:D_T-1_P5.08mm_Horizontal")
     )
     (path "/e483a1a3-bb43-4adf-8c54-28292661b80b"
@@
       (reference "Jac1") (unit 1) (value "Screw_Terminal_01x02") (footprint "TerminalBlock:TerminalBlock_bornier-2_P5.08mm")
     )
-    (path "/a3d8d232-73a6-4eab-be24-27abf5767e22"
-      (reference "Jdc1") (unit 1) (value "Barrel_Jack_MountingPin") (footprint "Connector_BarrelJack:BarrelJack_Horizontal")
+    (path "/dd9782b6-cb17-41e2-89ae-760613e6a0b3"
+      (reference "Jdc1") (unit 1) (value "Barrel_Jack_Switch") (footprint "Connector_BarrelJack:BarrelJack_CUI_PJ-102AH_Horizontal")
     )
     (path "/82371573-d06e-4132-9cab-402252dacf92"

Commit message: Fazendo a PCB
Parts:
- added Dwifi1: LED, LED_THT:LED_D3.0mm, symbol Device:LED
- added JP1: Jumper_2_Bridged, Jumper:jumper_10mm, symbol Jumper:Jumper_2_Bridged
- added Rwifi1: 260, Resistor_THT:R_Axial_DIN0207_L6.3mm_D2.5mm_P7.62mm_Horizontal, symbol Device:R
Connections:
- net +5V: now also JP1.2 (B); no longer Jpwr_sens1.1 (Pin_1), Jpwr_sens1.2 (Pin_2), Jpwr_sens1.3 (Pin_3), Jpwr_sens1.4 (Pin_4), Jpwr_sens1.5 (Pin_5), Jpwr_sens1.6 (Pin_6), Jpwr_sens1.7 (Pin_7), Jpwr_sens1.8 (Pin_8)
- net GND: now also Dwifi1.1 (K)
- net multiplex_A: now also U1.6 (GPIO12); no longer U1.4 (GPIO16)
- net multiplex_C: now also U1.4 (GPIO16); no longer U1.6 (GPIO12)
- net S4: now reaches Jsens1.5 (Pin_5), Umultiplex1.1 (X4)
- net S2: now reaches Jsens1.4 (Pin_4)
- net S2: now also Umultiplex1.15 (X2); no longer Umultiplex1.12 (X3)
- net S0: now reaches Umultiplex1.13 (X0)
- net S0: now also Jsens1.2 (Pin_2); no longer Jsens1.1 (Pin_1)
- net S1: now reaches Umultiplex1.14 (X1)
- net S1: now also Jsens1.3 (Pin_3); no longer Jsens1.2 (Pin_2)
- net S6: now reaches Umultiplex1.2 (X6)
- net S6: now also Jsens1.6 (Pin_6); no longer Jsens1.7 (Pin_7)
- net S5: now reaches Jsens1.8 (Pin_8)
- net S5: now also Umultiplex1.5 (X5); no longer Umultiplex1.4 (X7)
- net wifi_status: now reaches U1.17 (GPIO2)
- net wifi_status: now also Rwifi1.1
- new net: JP1.1 (A), Jpwr_sens1.1 (Pin_1), Jpwr_sens1.2 (Pin_2), Jpwr_sens1.3 (Pin_3), Jpwr_sens1.4 (Pin_4), Jpwr_sens1.5 (Pin_5), Jpwr_sens1.6 (Pin_6), Jpwr_sens1.7 (Pin_7), Jpwr_sens1.8 (Pin_8)
- new net: Dwifi1.2 (A), Rwifi1.2
- new net S3: Jsens1.1 (Pin_1), Umultiplex1.12 (X3)
- new net S7: Jsens1.7 (Pin_7), Umultiplex1.4 (X7)
- no-connect marks 9 -> 8
Other:
- note added: "Status"
- note removed: "NC_internal_led"
- note removed: "Steady State Status"
- moved on the sheet: Dss1, Jsens1, Jserial_com1, Jserial_power1, Rsens1, Rsens2, Rss1, Umultiplex1
