File: kicad/projeto/projeto.kicad_sch (KiCad schematic)
At the start: 43 parts, among them Q1 BTA16-600B, Q2 BTA16-600B, U1 ESP-12E, U3v3 LM1117-3.3

Commit message: Fazendo a PCB
Connections:
- net AC1: now also Jl2.2 (Pin_2); no longer Jl2.1 (Pin_1)
- net AC2: now also Jac1.1 (Pin_1); no longer Jac1.2 (Pin_2)
- net at F1.1: now also Jac1.2 (Pin_2); no longer Jac1.1 (Pin_1)
- net at Q2.2 (A2), Rtriac2.2: now also Jl2.1 (Pin_1); no longer Jl2.2 (Pin_2)
Other:
- moved on the sheet: Jac1, Jl2
Changed lines of the file:
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@@
     (pin "1")
   )
-  (symbol (lib_id "Connector:Screw_Terminal_01x02") (at 121.92 125.73 0) (mirror y) (unit 1)
+  (symbol (lib_id "Connector:Screw_Terminal_01x02") (at 121.92 128.27 180) (unit 1)
     (in_bom yes) (on_board yes) (fields_autoplaced)
     (property "Reference" "Jac1" (id 0) (at 121.92 119.38 0))
     (property "Value" "Screw_Terminal_01x02" (id 1) (at 121.92 121.92 0))
-    (property "Footprint" "TerminalBlock:TerminalBlock_bornier-2_P5.08mm" (id 2) (at 121.92 125.73 0)
-      (effects (font (size 1.27 1.27)) hide)
-    )
-    (property "Datasheet" "~" (id 3) (at 121.92 125.73 0)
+    (property "Footprint" "TerminalBlock:TerminalBlock_bornier-2_P5.08mm" (id 2) (at 121.92 128.27 0)
+      (effects (font (size 1.27 1.27)) hide)
+    )
+    (property "Datasheet" "~" (id 3) (at 121.92 128.27 0)
       (effects (font (size 1.27 1.27)) hide)
     )
@@
     (pin "2")
   )
-  (symbol (lib_id "Connector:Screw_Terminal_01x02") (at 53.34 158.75 90) (unit 1)
-    (in_bom yes) (on_board yes)
-    (property "Reference" "Jl2" (id 0) (at 52.07 152.4 90)
-      (effects (font (size 1.27 1.27)) (justify right))
-    )
-    (property "Value" "Screw_Terminal_01x02" (id 1) (at 52.07 154.94 90)
-      (effects (font (size 1.27 1.27)) (justify right))
-    )
-    (property "Footprint" "TerminalBlock:TerminalBlock_bornier-2_P5.08mm" (id 2) (at 53.34 158.75 0)
-      (effects (font (size 1.27 1.27)) hide)
-    )
-    (property "Datasheet" "~" (id 3) (at 53.34 158.75 0)
-      (effects (font (size 1.27 1.27)) hide)
-    )
+  (symbol (lib_id "Connector:Screw_Terminal_01x02") (at 55.88 158.75 270) (mirror x) (unit 1)
+    (in_bom yes) (on_board yes)
+    (property "Reference" "Jl2" (id 0) (at 48.26 152.4 90)
+      (effects (font (size 1.27 1.27)) (justify right))
+    )
+    (property "Value" "Screw_Terminal_01x02" (id 1) (at 66.04 154.94 90)
+      (effects (font (size 1.27 1.27)) (justify right))
+    )
+    (property "Footprint" "TerminalBlock:TerminalBlock_bornier-2_P5.08mm" (id 2) (at 55.88 158.75 0)
+      (effects (font (size 1.27 1.27)) hide)
+    )
+    (property "Datasheet" "~" (id 3) (at 55.88 158.75 0)
+      (effects (font (size 1.27 1.27)) hide)
+    )

Commit message: Fazendo a PCB
Parts:
- added Don1: LED, LED_THT:LED_D3.0mm, symbol Device:LED
- added JP2, JP3, JP4: Jumper_2_Bridged, Jumper:jumper_10mm, symbol Jumper:Jumper_2_Bridged
- added Ron1: 260, Resistor_THT:R_Axial_DIN0207_L6.3mm_D2.5mm_P7.62mm_Horizontal, symbol Device:R
- Udet_0: footprint Package_DIP:DIP-6_W7.62mm -> Package_DIP:DIP-6_W7.62mm_Socket_LongPads
- Uload1, Uload2: footprint Package_DIP:DIP-6_W7.62mm_LongPads -> Package_DIP:DIP-6_W7.62mm_Socket_LongPads
Connections:
- net +3V3: now also Ron1.1
- net AC1: now also JP4.1 (A); no longer D1.2 (A), D2.1 (K)
- net AC2: now also JP2.1 (A), JP3.1 (A); no longer D3.2 (A), D4.1 (K), Q2.1 (A1)
- net GND: now also Don1.1 (K)
- new net: D1.2 (A), D2.1 (K), JP4.2 (B)
- new net: Don1.2 (A), Ron1.2
- new net AC2': D3.2 (A), D4.1 (K), JP2.2 (B), JP3.2 (B), Q2.1 (A1)
Other:
- moved on the sheet: D1, D2, D3, D4, D5, Rz1, Rz2, Udet_0

Commit message: Fazendo a PCB
Connections:
- net det_0_intr: now also U1.7 (GPIO13); no longer U1.16 (GPIO15)
- net steady_state: now also U1.16 (GPIO15); no longer U1.7 (GPIO13)
Changed lines of the file:
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@@
     (effects (font (size 1.27 1.27)) (justify right bottom))
   )
-  (label "det_0_intr" (at 241.3 76.2 0)
+  (label "det_0_intr" (at 241.3 71.12 0)
     (effects (font (size 1.27 1.27)) (justify left bottom))
   )
@@
     (effects (font (size 1.27 1.27)) (justify left bottom))
   )
-  (label "steady_state" (at 241.3 71.12 0)
+  (label "steady_state" (at 241.3 76.2 0)
     (effects (font (size 1.27 1.27)) (justify left bottom))
   )

Commit message: Fazendo a PCB
Parts:
- added JP5, JP6, JP8, JP9: Jumper_2_Bridged, Jumper:jumper_10mm, symbol Jumper:Jumper_2_Bridged
- added JP7: Jumper_2_Bridged, symbol Jumper:Jumper_2_Bridged
Connections:
- net +3V3: now also JP5.1 (A); no longer Ron1.1, Rreset1.1, Rz2.1, SWexit1.1, U1.8 (VCC)
- net GND: now also JP6.2 (B); no longer U1.15 (GND)
- net drive_load_1: now also JP7.2 (B); no longer Rmoc1.2
- net drive_load_2: now also JP8.2 (B); no longer Rmoc2.2
- net 5v': now reaches JP1.1 (A), Jpwr_sens1.1 (Pin_1), Jpwr_sens1.2 (Pin_2), Jpwr_sens1.3 (Pin_3), Jpwr_sens1.4 (Pin_4), Jpwr_sens1.5 (Pin_5), Jpwr_sens1.6 (Pin_6), Jpwr_sens1.7 (Pin_7), Jpwr_sens1.8 (Pin_8)
- net AC1': now reaches D1.2 (A), D2.1 (K), JP4.2 (B)
- new net: JP7.1 (A), Rmoc1.2
- new net: JP8.1 (A), Rmoc2.2
- new net 3v3'1: JP5.2 (B), JP9.1 (A), Rz2.1, U1.8 (VCC)
- new net 3v3'2: JP9.2 (B), Ron1.1, Rreset1.1, SWexit1.1
- new net gnd': JP6.1 (A), U1.15 (GND)
Other:
- moved on the sheet: C1, C2, D1, D2, D3, D4, D5, Don1, Dss1, Dwifi1, F1, JP1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

Commit message: Fix PCB
Parts:
- JP7: footprint (none) -> Jumper:jumper_10mm
Connections:
- net 3v3'2: now also Rexit1.1; no longer SWexit1.1
- net GND: now also SWexit1.2; no longer Rexit1.2
- net exit_intr: now also Rexit1.2, SWexit1.1; no longer Rexit1.1, SWexit1.2
Other:
- moved on the sheet: Rexit1, SWexit1
Changed lines of the file:
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@@
   (junction (at 223.52 137.16) (diameter 0) (color 0 0 0 0)
   )
-  (junction (at 63.5 106.68) (diameter 0) (color 0 0 0 0)
-  )
   (junction (at 224.79 46.99) (diameter 0) (color 0 0 0 0)
   )
@@
   )
   (junction (at 223.52 139.7) (diameter 0) (color 0 0 0 0)
+  )
+  (junction (at 60.96 106.68) (diameter 0) (color 0 0 0 0)
   )
   (junction (at 110.49 57.15) (diameter 0) (color 0 0 0 0)
@@
     (stroke (width 0) (type default) (color 0 0 0 0))
   )
+  (wire (pts (xy 60.96 106.68) (xy 60.96 110.49))
+    (stroke (width 0) (type default) (color 0 0 0 0))
+  )
   (wire (pts (xy 72.39 45.72) (xy 74.93 45.72))
     (stroke (width 0) (type default) (color 0 0 0 0))
@@
     (stroke (width 0) (type default) (color 0 0 0 0))
   )
-  (wire (pts (xy 62.23 106.68) (xy 63.5 106.68))
-    (stroke (width 0) (type default) (color 0 0 0 0))
-  )
   (wire (pts (xy 72.39 58.42) (xy 74.93 58.42))
     (stroke (width 0) (type default) (color 0 0 0 0))
   )
+  (wire (pts (xy 60.96 106.68) (xy 62.23 106.68))
+    (stroke (width 0) (type default) (color 0 0 0 0))
+  )
+  (wire (pts (xy 59.69 106.68) (xy 60.96 106.68))
+    (stroke (width 0) (type default) (color 0 0 0 0))
+  )
   (wire (pts (xy 80.01 160.02) (xy 80.01 165.1))
     (stroke (width 0) (type default) (color 0 0 0 0))
@@
     (stroke (width 0) (type default) (color 0 0 0 0))
   )
-  (wire (pts (xy 63.5 106.68) (xy 63.5 110.49))
-    (stroke (width 0) (type default) (color 0 0 0 0))
-  )
   (wire (pts (xy 71.12 170.18) (xy 80.01 170.18))
     (stroke (width 0) (type default) (color 0 0 0 0))
@@
     (stroke (width 0) (type default) (color 0 0 0 0))
   )
-  (wire (pts (xy 63.5 106.68) (xy 64.77 106.68))
-    (stroke (width 0) (type default) (color 0 0 0 0))
-  )
   (wire (pts (xy 153.67 121.92) (xy 154.94 121.92))
     (stroke (width 0) (type default) (color 0 0 0 0))
@@
     (effects (font (size 1.27 1.27)) (justify right bottom))
   )
-  (label "exit_intr" (at 63.5 110.49 180)
-    (effects (font (size 1.27 1.27)) (justify right bottom))
+  (label "exit_intr" (at 60.96 110.49 0)
+    (effects (font (size 1.27 1.27)) (justify left bottom))
   )
   (label "multiplex_C" (at 243.84 78.74 0)
@@
     (pin "8")
   )
-  (symbol (lib_id "Switch:SW_Push") (at 57.15 106.68 0) (unit 1)
-    (in_bom yes) (on_board yes) (fields_autoplaced)
-    (property "Reference" "SWexit1" (id 0) (at 57.15 99.06 0))
-    (property "Value" "SW_Push" (id 1) (at 57.15 101.6 0))
-    (property "Footprint" "Button_Switch_THT:SW_PUSH_6mm" (id 2) (at 57.15 101.6 0)
-      (effects (font (size 1.27 1.27)) hide)
-    )
-    (property "Datasheet" "~" (id 3) (at 57.15 101.6 0)
+  (symbol (lib_id "Switch:SW_Push") (at 67.31 106.68 0) (unit 1)
+    (in_bom yes) (on_board yes) (fields_autoplaced)
+    (property "Reference" "SWexit1" (id 0) (at 67.31 99.06 0))
+    (property "Value" "SW_Push" (id 1) (at 67.31 101.6 0))
+    (property "Footprint" "Button_Switch_THT:SW_PUSH_6mm" (id 2) (at 67.31 101.6 0)
+      (effects (font (size 1.27 1.27)) hide)
+    )
+    (property "Datasheet" "~" (id 3) (at 67.31 101.6 0)
       (effects (font (size 1.27 1.27)) hide)
     )
@@
     (property "Reference" "JP7" (id 0) (at 102.87 118.11 0))
     (property "Value" "Jumper_2_Bridged" (id 1) (at 102.87 120.65 0))
-    (property "Footprint" "" (id 2) (at 102.87 124.46 0)
+    (property "Footprint" "Jumper:jumper_10mm" (id 2) (at 102.87 124.46 0)
       (effects (font (size 1.27 1.27)) hide)
     )
@@
     (pin "2")
   )
-  (symbol (lib_id "Device:R") (at 68.58 106.68 90) (unit 1)
-    (in_bom yes) (on_board yes) (fields_autoplaced)
-    (property "Reference" "Rexit1" (id 0) (at 68.58 100.33 90))
-    (property "Value" "10K" (id 1) (at 68.58 102.87 90))
-    (property "Footprint" "Resistor_THT:R_Axial_DIN0207_L6.3mm_D2.5mm_P7.62mm_Horizontal" (id 2) (at 68.58 108.458 90)
-      (effects (font (size 1.27 1.27)) hide)
-    )
-    (property "Datasheet" "~" (id 3) (at 68.58 106.68 0)
-      (effects (font (size 1.27 1.27)) hide)
-    )
+  (symbol (lib_id "Device:R") (at 55.88 106.68 90) (unit 1)
+    (in_bom yes) (on_board yes) (fields_autoplaced)
+    (property "Reference" "Rexit1" (id 0) (at 55.88 100.33 90))
+    (property "Value" "10K" (id 1) (at 55.88 102.87 90))
+    (property "Footprint" "Resistor_THT:R_Axial_DIN0207_L6.3mm_D2.5mm_P7.62mm_Horizontal" (id 2) (at 55.88 108.458 90)
+      (effects (font (size 1.27 1.27)) hide)
+    )
+    (property "Datasheet" "~" (id 3) (at 55.88 106.68 0)
+      (effects (font (size 1.27 1.27)) hide)
+    )
