File: kicad/projeto/projeto.kicad_pcb (KiCad board)
At the start: 2 copper layers, 40 parts, among them Q1 BTA16-600B, Q2 BTA16-600B, U1 ESP-12E, U3v3 LM1117-3.3

Commit message: Fazendo a PCB
Parts:
- added Dwifi1: LED, LED_THT:LED_D3.0mm, F.Cu at (94.0, 125.7)
- added JP1: Jumper_2_Bridged, Jumper:jumper_10mm, F.Cu at (228.6, 106.7)
- added Rwifi1: 260, Resistor_THT:R_Axial_DIN0207_L6.3mm_D2.5mm_P7.62mm_Horizontal, F.Cu at (83.1, 125.0)
- C1, C2, Jdc1, Jpwr_sens1, Jpwr_sens2, Jsens1, Jserial_power1, Rsens1, Rsens2, U3v3, Umultiplex1: moved to B.Cu
- moved Jserial_power1 196.3 mm to (234.9, 132.1), turned to 180 degrees
- moved Jdc1 195.0 mm to (232.4, 114.3)
- moved C1 177.7 mm to (226.1, 122.0), turned to -90 degrees
- moved U3v3 165.7 mm to (217.0, 114.3), turned to 0 degrees
- moved C2 153.5 mm to (214.6, 122.0), turned to -90 degrees
- moved Umultiplex1 90.1 mm to (203.2, 87.6)
- moved Jpwr_sens1 80.7 mm to (229.9, 82.5), turned to 180 degrees
- moved D1 77.5 mm to (141.0, 57.8)
- moved D2 77.5 mm to (148.6, 52.7)
- moved D3 77.5 mm to (141.0, 69.8)
- moved D4 77.5 mm to (148.6, 74.9)
- moved D5 77.5 mm to (133.3, 57.8)
- moved Rz1 77.5 mm to (135.9, 64.1)
- moved Rz2 77.5 mm to (125.7, 80.6)
- moved Udet_0 77.5 mm to (128.3, 62.9)
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Connections:
- net Net-(Jsens1-Pad5) renamed /S4
- Jpwr_sens1 pad 1: +5V -> Net-(JP1-Pad1)
- Jpwr_sens1 pad 2: +5V -> Net-(JP1-Pad1)
- Jpwr_sens1 pad 3: +5V -> Net-(JP1-Pad1)
- Jpwr_sens1 pad 4: +5V -> Net-(JP1-Pad1)
- Jpwr_sens1 pad 5: +5V -> Net-(JP1-Pad1)
- Jpwr_sens1 pad 6: +5V -> Net-(JP1-Pad1)
- Jpwr_sens1 pad 7: +5V -> Net-(JP1-Pad1)
- Jpwr_sens1 pad 8: +5V -> Net-(JP1-Pad1)
- Jsens1 pad 1: Net-(Jsens1-Pad1) -> /S3
- Jsens1 pad 2: Net-(Jsens1-Pad2) -> /S0
- Jsens1 pad 3: Net-(Jsens1-Pad3) -> /S1
- Jsens1 pad 4: Net-(Jsens1-Pad4) -> /S2
- Jsens1 pad 6: Net-(Jsens1-Pad6) -> /S6
- Jsens1 pad 7: Net-(Jsens1-Pad7) -> /S7
- Jsens1 pad 8: Net-(Jsens1-Pad8) -> /S5
- U1 pad 17: unconnected-(U1-Pad17) -> /wifi_status
- Umultiplex1 pad 12: Net-(Jsens1-Pad4) -> /S3
- Umultiplex1 pad 13: Net-(Jsens1-Pad1) -> /S0
- Umultiplex1 pad 14: Net-(Jsens1-Pad2) -> /S1
- Umultiplex1 pad 15: Net-(Jsens1-Pad3) -> /S2
- Umultiplex1 pad 2: Net-(Jsens1-Pad7) -> /S6
- Umultiplex1 pad 4: Net-(Jsens1-Pad8) -> /S7
- Umultiplex1 pad 5: Net-(Jsens1-Pad6) -> /S5
Routing:
- net /AC2: track 74.1 -> 0.00 mm
- net Net-(Jl1-Pad2): track 72.2 -> 0.00 mm
- net /AC1: track 71.9 -> 0.00 mm
- net GND: track 194.1 -> 127.0 mm
- net +3V3: track 113.5 -> 60.8 mm
- net /S3: track 0.00 -> 45.1 mm
- net /S0: track 0.00 -> 40.0 mm
- net /S1: track 0.00 -> 34.9 mm
- net Net-(Q1-Pad3): track 34.7 -> 0.00 mm
- net /multiplex_out: track 34.0 -> 3.81 mm
- net /S2: track 0.00 -> 29.8 mm
- net Net-(JP1-Pad1): track 0.00 -> 24.7 mm
- net /multiplex_C: track 22.6 -> 0.00 mm
- net /multiplex_B: track 21.6 -> 0.00 mm
- net /multiplex_A: track 20.7 -> 0.03 mm
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Other:
- board outline added: 209.5 x 138.4 mm
- board text added: "+5V"
- board text added: "gnd"

Commit message: Fazendo a PCB
Parts:
- F1, Jac1, Jl1, Jl2, Q1, Q2, Rmoc1, Rmoc2, Rtriac1, Rtriac2, Uload1, Uload2: moved to B.Cu
- moved Jl2 109.2 mm to (238.8, 36.8), turned to -90 degrees
- moved D1 82.8 mm to (59.6, 42.5)
- moved D2 82.8 mm to (67.2, 37.5)
- moved D3 82.8 mm to (59.6, 54.6)
- moved D4 82.8 mm to (67.2, 59.7)
- moved D5 82.8 mm to (51.9, 42.5)
- moved Rz1 82.8 mm to (54.5, 48.9)
- moved Rz2 82.8 mm to (44.3, 65.4)
- moved Udet_0 82.8 mm to (46.8, 47.6)
- moved Q2 73.7 mm to (157.5, 33.0), turned to 180 degrees
- moved Rmoc2 44.0 mm to (152.4, 55.9), turned to 180 degrees
- moved Rtriac2 40.9 mm to (147.3, 43.2)
- moved Uload2 33.1 mm to (156.2, 48.2), turned to -90 degrees
- moved Uload1 28.0 mm to (196.9, 48.2)
- moved Rmoc1 25.6 mm to (193.0, 55.9)
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Connections:
- Jac1 pad 1: Net-(F1-Pad1) -> /AC2
- Jac1 pad 2: /AC2 -> Net-(F1-Pad1)
- Jl2 pad 1: /AC1 -> Net-(Jl2-Pad1)
- Jl2 pad 2: Net-(Jl2-Pad2) -> /AC1
- Q2 pad 2: Net-(Jl2-Pad2) -> Net-(Jl2-Pad1)
- Rtriac2 pad 2: Net-(Jl2-Pad2) -> Net-(Jl2-Pad1)
- U1 pad 4: /multiplex_A -> /multiplex_C
- U1 pad 6: /multiplex_C -> /multiplex_A
Routing:
- net Net-(Jl1-Pad2): track 0.00 -> 77.0 mm
- net /AC2: track 0.00 -> 59.3 mm
- net GND: track 127.0 -> 171.1 mm
- net /AC1: track 0.00 -> 40.4 mm
- net Net-(Q1-Pad3): track 0.00 -> 19.3 mm
- net Net-(Q2-Pad3): track 0.00 -> 19.3 mm
- net Net-(F1-Pad1): track 0.00 -> 17.8 mm
- net Net-(Rtriac1-Pad1): track 0.00 -> 11.7 mm
- net Net-(Rtriac2-Pad1): track 0.00 -> 11.7 mm
- net Net-(Rmoc1-Pad1): track 0.00 -> 3.83 mm
- net Net-(Rmoc2-Pad1): track 0.00 -> 3.81 mm
- net Net-(Rsens1-Pad1): track 22.1 -> 20.6 mm
- net +3V3: track 60.8 -> 59.6 mm
- net /S3: track 45.1 -> 44.5 mm
- net /S6: track 13.6 -> 13.0 mm
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
Commit message: Fazendo a PCB
Parts:
- added ?: , , F.Cu at (241.3, 156.2)
- added Don1: LED, LED_THT:LED_D3.0mm, F.Cu at (83.8, 118.1)
- added JP2: Jumper_2_Bridged, Jumper:jumper_10mm, B.Cu at (208.2, 61.0)
- added JP3: Jumper_2_Bridged, Jumper:jumper_10mm, B.Cu at (208.2, 58.4)
- added JP4: Jumper_2_Bridged, Jumper:jumper_10mm, B.Cu at (179.1, 50.8)
- added REF**: MountingHole_3mm_Pad, MountingHole:MountingHole_3mm_Pad, F.Cu at (241.3, 156.2)
- added REF**: MountingHole_3mm_Pad, MountingHole:MountingHole_3mm_Pad, F.Cu at (241.3, 36.8)
- added Ron1: 260, Resistor_THT:R_Axial_DIN0207_L6.3mm_D2.5mm_P7.62mm_Horizontal, F.Cu at (73.0, 117.4)
- D1, D2, D3, D4, D5, Rz1, Rz2: moved to B.Cu
- Udet_0: footprint Package_DIP:DIP-6_W7.62mm -> Package_DIP:DIP-6_W7.62mm_Socket_LongPads; moved to B.Cu
- Uload1, Uload2: footprint Package_DIP:DIP-6_W7.62mm_LongPads -> Package_DIP:DIP-6_W7.62mm_Socket_LongPads
- moved Udet_0 138.0 mm to (181.6, 77.5)
- moved Rz2 134.3 mm to (176.5, 88.9), turned to 0 degrees
- moved D1 129.8 mm to (186.7, 68.6)
- moved D5 124.5 mm to (171.4, 77.5), turned to 0 degrees
- moved Rz1 119.3 mm to (171.4, 72.4)
- moved D2 117.4 mm to (181.6, 63.5)
- moved D3 112.8 mm to (171.4, 68.6), turned to 90 degrees
- moved D4 109.4 mm to (176.5, 63.5), turned to -90 degrees
- moved U1 62.3 mm to (167.6, 147.3)
- moved Rmoc1 36.4 mm to (208.3, 88.9)
- moved Rmoc2 33.1 mm to (154.9, 88.9)
- moved Uload1 30.5 mm to (205.7, 77.5)
- moved Uload2 29.5 mm to (152.4, 77.5)
- moved Rtriac1 23.3 mm to (196.8, 64.8)
- moved Rtriac2 20.4 mm to (146.1, 63.5)
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Connections:
- D1 pad 2: /AC1 -> Net-(D1-Pad2)
- D2 pad 1: /AC1 -> Net-(D1-Pad2)
- D3 pad 2: /AC2 -> /AC2'
- D4 pad 1: /AC2 -> /AC2'
- Q2 pad 1: /AC2 -> /AC2'
Routing:
- net Net-(Jl2-Pad1): track 0.00 -> 111.0 mm
- net /AC1: track 40.4 -> 102.9 mm
- net /AC2': track 0.00 -> 53.5 mm
- net Net-(D1-Pad1): track 0.00 -> 31.3 mm
- net GND: track 171.1 -> 187.8 mm
- net Net-(Rz1-Pad1): track 1.13 -> 16.3 mm
- net Net-(D2-Pad2): track 0.00 -> 13.2 mm
- net Net-(Q1-Pad3): track 19.3 -> 31.4 mm
- net Net-(D1-Pad2): track 0.00 -> 9.48 mm
- net Net-(Q2-Pad3): track 19.3 -> 27.2 mm
- net Net-(Rtriac1-Pad1): track 11.7 -> 19.4 mm
- net Net-(Rtriac2-Pad1): track 11.7 -> 18.8 mm
- net /AC2: track 59.3 -> 66.4 mm
- net Net-(D5-Pad2): track 0.02 -> 5.08 mm
- net Net-(Jl1-Pad2): track 77.0 -> 81.4 mm
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Other:
- board size 209.5 x 138.4 mm -> 209.6 x 138.4 mm
- board text added: "Back"
- board text added: "Front"
- board text removed: "Checar a tensão do cp2102. Se mandar 5V,"
- board text removed: "Colocar um divisor de tensão e mais 2 pinos"

Commit message: Fazendo a PCB
Parts:
- Don1, Dss1, Dwifi1, Jserial_com1, Ren1, Rexit1, Ron1, Rreset1, Rss1, Rwifi1, SWexit1, SWreset1: moved to B.Cu
- moved SWexit1 83.0 mm to (132.8, 136.6), turned to 90 degrees
- moved SWreset1 82.7 mm to (132.8, 149.3), turned to 90 degrees
- moved Rexit1 80.0 mm to (137.2, 137.2), turned to 90 degrees
- moved Jserial_com1 76.5 mm to (167.6, 147.3), turned to 180 degrees
- moved Ren1 75.1 mm to (195.6, 146.8), turned to 0 degrees
- moved Rreset1 74.7 mm to (137.2, 142.3), turned to -90 degrees
- moved Ron1 69.8 mm to (142.2, 108.5), turned to 180 degrees
- moved Rwifi1 59.4 mm to (142.2, 121.2), turned to 180 degrees
- moved Don1 45.5 mm to (128.3, 108.5)
- moved Rss1 40.4 mm to (142.2, 114.9), turned to 180 degrees
- moved Dwifi1 37.7 mm to (128.3, 121.2)
- moved Dss1 30.2 mm to (128.3, 114.9)
- moved U1 12.7 mm to (180.3, 147.3)
- moved D1 2.54 mm to (186.7, 71.1)
- moved D2 2.54 mm to (181.6, 66.0)
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Connections:
- U1 pad 16: /det_0_intr -> /steady_state
- U1 pad 7: /steady_state -> /det_0_intr
Routing:
- net /det_0_intr: track 0.00 -> 56.2 mm
- net GND: track 187.8 -> 239.8 mm
- net /multiplex_A: track 0.00 -> 29.9 mm
- net /multiplex_B: track 0.00 -> 29.8 mm
- net /multiplex_C: track 0.00 -> 28.8 mm
- net /multiplex_out: track 3.81 -> 29.9 mm
- net +3V3: track 59.3 -> 84.7 mm
- net /exit_intr: track 0.79 -> 24.6 mm
- net /reset: track 1.20 -> 11.1 mm
- net /Enable: track 0.00 -> 7.64 mm
- net /S3: track 44.5 -> 38.0 mm
- net /Serial_rx: track 0.00 -> 5.72 mm
- net Net-(Rmoc2-Pad1): track 0.02 -> 5.65 mm
- net Net-(Rmoc1-Pad1): track 0.00 -> 5.62 mm
- net /Serial_tx: track 0.00 -> 5.50 mm
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Other:
- board size 209.6 x 138.4 mm -> 209.6 x 127 mm
- board text added: "12"
- board text added: "I/O"

Commit message: Fazendo a PCB
Parts:
- removed ?: , 
- added JP5: Jumper_2_Bridged, Jumper:jumper_10mm, B.Cu at (201.9, 133.3)
- added JP6: Jumper_2_Bridged, Jumper:jumper_10mm, B.Cu at (191.9, 137.2)
- added JP7: Jumper_2_Bridged, Jumper:jumper_10mm, B.Cu at (167.6, 132.2)
- added JP8: Jumper_2_Bridged, Jumper:jumper_10mm, B.Cu at (163.8, 132.2)
- added JP9: Jumper_2_Bridged, Jumper:jumper_10mm, B.Cu at (170.2, 128.3)
- added REF**: MountingHole_3mm_Pad, MountingHole:MountingHole_3mm_Pad, F.Cu at (133.3, 156.2)
- added REF**: MountingHole_3mm_Pad, MountingHole:MountingHole_3mm_Pad, F.Cu at (133.3, 39.4)
- moved Don1 16.5 mm to (144.8, 108.5)
- moved Dss1 16.5 mm to (144.8, 114.9)
- moved Dwifi1 16.5 mm to (144.8, 121.2)
- moved Rexit1 16.5 mm to (153.7, 137.2)
- moved Ron1 16.5 mm to (158.8, 108.5)
- moved Rreset1 16.5 mm to (153.7, 142.3)
- moved Rss1 16.5 mm to (158.8, 114.9)
- moved Rwifi1 16.5 mm to (158.8, 121.2)
- moved SWexit1 16.5 mm to (149.3, 136.6)
- moved SWreset1 16.5 mm to (149.3, 149.3)
- moved Rz2 10.2 mm to (186.7, 91.4), turned to 180 degrees
- moved REF** 5.08 mm to (246.4, 156.2)
- moved REF** 5.08 mm to (246.4, 39.4)
- moved Rsens2 3.81 mm to (199.4, 129.5)
- moved Rsens1 3.81 mm to (207.0, 125.7)
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Connections:
- net Net-(D1-Pad2) renamed /AC1'
- net Net-(JP1-Pad1) renamed /5v'
- Rmoc1 pad 2: /drive_load_1 -> Net-(Rmoc1-Pad2)
- Rmoc2 pad 2: /drive_load_2 -> Net-(Rmoc2-Pad2)
- Ron1 pad 1: +3V3 -> /3v3'2
- Rreset1 pad 1: +3V3 -> /3v3'2
- Rz2 pad 1: +3V3 -> /3v3'1
- SWexit1 pad 1: +3V3 -> /3v3'2
- U1 pad 15: GND -> /gnd'
- U1 pad 8: +3V3 -> /3v3'1
Routing:
- net /3v3'1: track 0.00 -> 86.4 mm
- net GND: track 239.8 -> 317.3 mm
- net Net-(Rmoc1-Pad2): track 0.00 -> 75.7 mm
- net Net-(Rmoc2-Pad2): track 0.00 -> 51.1 mm
- net /3v3'2: track 0.00 -> 49.9 mm
- net /reset: track 11.1 -> 49.0 mm
- net /steady_state: track 0.00 -> 36.5 mm
- net /det_0_intr: track 56.2 -> 88.7 mm
- net /wifi_status: track 0.00 -> 31.2 mm
- net /exit_intr: track 24.6 -> 47.8 mm
- net /gnd': track 0.00 -> 19.9 mm
- net /drive_load_2: track 0.00 -> 11.6 mm
- net /drive_load_1: track 0.00 -> 6.17 mm
- net /multiplex_A: track 29.9 -> 33.2 mm
- net /multiplex_C: track 28.8 -> 32.1 mm
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Other:
- board size 209.6 x 127 mm -> 123.2 x 127 mm
- board text added: "GND"
- board text added: "S0"
- board text added: "S1"
- board text added: "S2"
- board text added: "S3"
- board text added: "S4"
- board text added: "S5"
- board text added: "S6"
- board text added: "S7"
- board text removed: "12"
- board text removed: "Back"
- board text removed: "Front"

Commit message: Fazendo a PCB
Parts:
- moved Rreset1 5.67 mm to (153.7, 136.6)
- moved SWreset1 5.67 mm to (149.3, 143.7)
- moved Don1 5.67 mm to (144.8, 102.9)
- moved Dss1 5.67 mm to (144.8, 109.2)
- moved Dwifi1 5.67 mm to (144.8, 115.6)
- moved Ron1 5.67 mm to (158.8, 102.9)
- moved Rss1 5.67 mm to (158.8, 109.2)
- moved Rwifi1 5.67 mm to (158.8, 115.6)
- moved Rexit1 5.67 mm to (153.7, 131.5)
- moved SWexit1 5.67 mm to (149.3, 131.0)
Routing:
- net /3v3'2: track 49.9 -> 56.0 mm
- net /wifi_status: track 31.2 -> 36.9 mm
- net /steady_state: track 36.5 -> 42.2 mm
- net /reset: track 49.0 -> 48.1 mm
- net Net-(Rmoc2-Pad2): track 51.1 -> 50.3 mm
